File: sDB.kicad_pcb (KiCad board)
At the start: 2 copper layers, 18 x 16.5 mm, 11 parts, among them J1 USB_C_Receptacle_USB2.0, J2 Conn_01x04

Commit message: remove logo
Parts:
- removed G***: LOGO, custom_parts:elmo

Commit message: add pinout labels
Other:
- board text added: "D+"
- board text added: "D-"
- board text added: "GND"
- board text added: "V+"
