File: fab/sDB_panel.kicad_pcb (KiCad board)
At the start: 2 copper layers, 48 x 35 mm, 152 parts, among them J1 USB_C_Receptacle_USB2.0, J2 Conn_01x04

Commit message: remove logo
Parts:
- removed G*** (x4): LOGO, custom_parts:elmo

Commit message: add pinout labels
Other:
- board text added: "D+"
- board text added: "D-"
- board text added: "GND"
- board text added: "V+"
